File: pcb/kicad/processor.kicad_sch (KiCad schematic)
At the start: 26 parts, among them J301 TagConnect_TC2030, U301 STM32F401RBTx, Y301 16MHz

Commit message: Add part numbers to components for ordering.
Parts:
- C4: Part Number (none) -> CC0805JRX7R9BB104
- C4: Part Number (none) -> CC0805KKX7R7BB105
- C4: Part Number (none) -> C0805C475M4RACTU
- C4: Part Number (none) -> C0805C100M4GACTU
- D301, D302, D303, D304, D305: Part Number (none) -> PESD3V3L1BA,115
- R3: Part Number (none) -> CRCW08050000Z0EC
- R3: Part Number (none) -> CMP0805AFX-49R9ELF
- R3: Part Number (none) -> AC0805FR-0710K5L
- U301: Part Number (none) -> STM32F401RBT6TR; Supplier Link (none) -> https://www.digikey.de/en/products/detail/stmicroelectronic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
- Y301: Supplier Link (none) -> https://www.digikey.com/en/products/detail/raltron-electron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
Changed lines of the file:
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@@
+      (effects (font (size 1.27 1.27)) hide)
+    )
+    (property "Supplier Link" "" (at 69.85 60.96 0)
+      (effects (font (size 1.27 1.27)) hide)
+    )
+    (property "Part Number" "CC0805JRX7R9BB104" (at 69.85 60.96 0)
       (effects (font (size 1.27 1.27)) hide)
     )
@@
       (effects (font (size 1.27 1.27)) hide)
     )
+    (property "Supplier Link" "" (at 43.18 60.96 0)
+      (effects (font (size 1.27 1.27)) hide)
+    )
+    (property "Part Number" "CC0805JRX7R9BB104" (at 43.18 60.96 0)
+      (effects (font (size 1.27 1.27)) hide)
+    )
     (pin "1")
     (pin "2")
@@
       (effects (font (size 1.27 1.27)) hide)
     )
+    (property "Supplier Link" "" (at 91.44 92.71 0)
+      (effects (font (size 1.27 1.27)) hide)
+    )
+    (property "Part Number" "CRCW08050000Z0EC" (at 91.44 92.71 0)
+      (effects (font (size 1.27 1.27)) hide)
+    )
     (pin "1")
     (pin "2")
@@
       (effects (font (size 1.27 1.27)) hide)
     )
+    (property "Supplier Link" "" (at 58.42 74.93 0)
+      (effects (font (size 1.27 1.27)) hide)
+    )
+    (property "Part Number" "CC0805KKX7R7BB105" (at 58.42 74.93 0)
+      (effects (font (size 1.27 1.27)) hide)
+    )
     (pin "1")
     (pin "2")
@@
     )
     (property "Datasheet" "~" (at 95.25 60.96 0)
+      (effects (font (size 1.27 1.27)) hide)
+    )
+    (property "Supplier Link" "" (at 95.25 60.96 0)
+      (effects (font (size 1.27 1.27)) hide)
+    )
+    (property "Part Number" "CC0805JRX7R9BB104" (at 95.25 60.96 0)
       (effects (font (size 1.27 1.27)) hide)
     )
@@
       (effects (font (size 1.27 1.27)) hide)
     )
-    (property "Datasheet" "" (at 71.12 163.83 0)
+    (property "Datasheet" "PESD3V3L1BA" (at 71.12 163.83 0)
+      (effects (font (size 1.27 1.27)) hide)
+    )
+    (property "Supplier Link" "" (at 71.12 163.83 0)
+      (effects (font (size 1.27 1.27)) hide)
+    )
+    (property "Part Number" "PESD3V3L1BA,115" (at 71.12 163.83 0)
       (effects (font (size 1.27 1.27)) hide)
     )
@@
     )
     (property "Datasheet" "https://www.st.com/resource/en/datasheet/stm32f401rb.pdf" (at 213.36 91.44 0)
+      (effects (font (size 1.27 1.27)) hide)
+    )
+    (property "Part Number" "STM32F401RBT6TR" (at 213.36 91.44 0)
+      (effects (font (size 1.27 1.27)) hide)
+    )
+    (property "Supplier Link" "https://www.digikey.de/en/products/detail/stmicroelectronics/STM32F401RBT6TR/5268280" (at 213.36 91.44 0)
       (effects (font (size 1.27 1.27)) hide)
     )
@@
       (effects (font (size 1.27 1.27)) hide)
     )
+    (property "Supplier Link" "" (at 57.15 60.96 0)
+      (effects (font (size 1.27 1.27)) hide)
+    )
+    (property "Part Number" "CC0805JRX7R9BB104" (at 57.15 60.96 0)
+      (effects (font (size 1.27 1.27)) hide)
+    )
     (pin "1")
     (pin "2")
@@
     )
     (property "Datasheet" "~" (at 107.95 60.96 0)
+      (effects (font (size 1.27 1.27)) hide)
+    )
+    (property "Supplier Link" "" (at 107.95 60.96 0)
+      (effects (font (size 1.27 1.27)) hide)
+    )
+    (property "Part Number" "C0805C475M4RACTU" (at 107.95 60.96 0)
       (effects (font (size 1.27 1.27)) hide)
     )
@@
       (effects (font (size 1.27 1.27)) hide)
     )
+    (property "Supplier Link" "" (at 101.6 156.21 0)
+      (effects (font (size 1.27 1.27)) hide)
+    )
+    (property "Part Number" "CMP0805AFX-49R9ELF" (at 101.6 156.21 0)
+      (effects (font (size 1.27 1.27)) hide)
+    )
     (pin "1")
     (pin "2")
@@
       (effects (font (size 1.27 1.27)) hide)
     )
-    (property "Datasheet" "" (at 78.74 163.83 0)
+    (property "Datasheet" "PESD3V3L1BA" (at 78.74 163.83 0)
+      (effects (font (size 1.27 1.27)) hide)
+    )
+    (property "Supplier Link" "" (at 78.74 163.83 0)
+      (effects (font (size 1.27 1.27)) hide)
+    )
+    (property "Part Number" "PESD3V3L1BA,115" (at 78.74 163.83 0)
       (effects (font (size 1.27 1.27)) hide)
     )
@@
     )
     (property "Datasheet" "~" (at 116.84 163.83 0)
+      (effects (font (size 1.27 1.27)) hide)
+    )
+    (property "Supplier Link" "" (at 116.84 163.83 0)
+      (effects (font (size 1.27 1.27)) hide)
+    )
+    (property "Part Number" "CC0805JRX7R9BB104" (at 116.84 163.83 0)
       (effects (font (size 1.27 1.27)) hide)
     )
@@
       (effects (font (size 1.27 1.27)) hide)
     )
-    (property "Datasheet" "" (at 63.5 163.83 0)
+    (property "Datasheet" "PESD3V3L1BA" (at 63.5 163.83 0)
+      (effects (font (size 1.27 1.27)) hide)
+    )
+    (property "Supplier Link" "" (at 63.5 163.83 0)
+      (effects (font (size 1.27 1.27)) hide)
+    )
+    (property "Part Number" "PESD3V3L1BA,115" (at 63.5 163.83 0)
       (effects (font (size 1.27 1.27)) hide)
     )
@@
       (effects (font (size 1.27 1.27)) hide)
     )
+    (property "Supplier Link" "" (at 101.6 153.67 0)
+      (effects (font (size 1.27 1.27)) hide)
+    )
+    (property "Part Number" "CMP0805AFX-49R9ELF" (at 101.6 153.67 0)
+      (effects (font (size 1.27 1.27)) hide)
+    )
     (pin "1")
     (pin "2")
@@
     )
     (property "Datasheet" "~" (at 173.99 55.88 0)
+      (effects (font (size 1.27 1.27)) hide)
+    )
+    (property "Supplier Link" "" (at 173.99 55.88 0)
+      (effects (font (size 1.27 1.27)) hide)
+    )
+    (property "Part Number" "AC0805FR-0710K5L" (at 173.99 55.88 0)
       (effects (font (size 1.27 1.27)) hide)
     )
@@
       (effects (font (size 1.27 1.27)) hide)
     )
+    (property "Supplier Link" "" (at 46.99 151.13 0)
+      (effects (font (size 1.27 1.27)) hide)
+    )
     (pin "1")
     (pin "2")
@@
       (effects (font (size 1.27 1.27)) hide)
     )
+    (property "Supplier Link" "" (at 101.6 151.13 0)
+      (effects (font (size 1.27 1.27)) hide)
+    )
+    (property "Part Number" "CMP0805AFX-49R9ELF" (at 101.6 151.13 0)
+      (effects (font (size 1.27 1.27)) hide)
+    )
     (pin "1")
     (pin "2")
@@
     )
     (property "Datasheet" "~" (at 74.93 97.79 0)
+      (effects (font (size 1.27 1.27)) hide)
+    )
+    (property "Supplier Link" "" (at 74.93 97.79 0)
+      (effects (font (size 1.27 1.27)) hide)
+    )
+    (property "Part Number" "C0805C100M4GACTU" (at 74.93 97.79 0)
       (effects (font (size 1.27 1.27)) hide)
     )
@@
       (effects (font (size 1.27 1.27)) hide)
     )
-    (property "Datasheet" "" (at 86.36 163.83 0)
+    (property "Datasheet" "PESD3V3L1BA" (at 86.36 163.83 0)
+      (effects (font (size 1.27 1.27)) hide)
+    )
+    (property "Supplier Link" "" (at 86.36 163.83 0)
+      (effects (font (size 1.27 1.27)) hide)
+    )
+    (property "Part Number" "PESD3V3L1BA,115" (at 86.36 163.83 0)
       (effects (font (size 1.27 1.27)) hide)
     )
@@
       (effects (font (size 1.27 1.27)) hide)
     )
+    (property "Supplier Link" "" (at 43.18 74.93 0)
+      (effects (font (size 1.27 1.27)) hide)
+    )
+    (property "Part Number" "CC0805JRX7R9BB104" (at 43.18 74.93 0)
+      (effects (font (size 1.27 1.27)) hide)
+    )
     (pin "1")
     (pin "2")
@@
       (effects (font (size 1.27 1.27)) hide)
     )
+    (property "Supplier Link" "" (at 82.55 60.96 0)
+      (effects (font (size 1.27 1.27)) hide)
+    )
+    (property "Part Number" "CC0805JRX7R9BB104" (at 82.55 60.96 0)
+      (effects (font (size 1.27 1.27)) hide)
+    )
     (pin "1")
     (pin "2")
@@
       (effects (font (size 1.27 1.27)) hide)
     )
+    (property "Supplier Link" "" (at 43.18 43.18 0)
+      (effects (font (size 1.27 1.27)) hide)
+    )
+    (property "Part Number" "C0805C475M4RACTU" (at 43.18 43.18 0)
+      (effects (font (size 1.27 1.27)) hide)
+    )
     (pin "1")
     (pin "2")
@@
     )
     (property "Part Number" "RH100-16.000-8-2020-TR" (at 62.23 92.71 0)
+      (effects (font (size 1.27 1.27)) hide)
+    )
+    (property "Supplier Link" "https://www.digikey.com/en/products/detail/raltron-electronics/RH100-16-000-8-2020-TR/15963324" (at 62.23 92.71 0)
       (effects (font (size 1.27 1.27)) hide)
     )
@@
       (effects (font (size 1.27 1.27)) hide)
     )
+    (property "Supplier Link" "" (at 44.45 97.79 0)
+      (effects (font (size 1.27 1.27)) hide)
+    )
+    (property "Part Number" "C0805C100M4GACTU" (at 44.45 97.79 0)
+      (effects (font (size 1.27 1.27)) hide)
+    )
     (pin "1")
     (pin "2")
@@
     )
     (property "Datasheet" "~" (at 101.6 146.05 0)
+      (effects (font (size 1.27 1.27)) hide)
+    )
+    (property "Supplier Link" "" (at 101.6 146.05 0)
+      (effects (font (size 1.27 1.27)) hide)
+    )
+    (property "Part Number" "CMP0805AFX-49R9ELF" (at 101.6 146.05 0)
       (effects (font (size 1.27 1.27)) hide)
     )
@@
       (effects (font (size 1.27 1.27)) hide)
     )
-    (property "Datasheet" "" (at 55.88 163.83 0)
-      (effects (font (size 1.27 1.27)) hide)
-    )
+    (property "Datasheet" "PESD3V3L1BA" (at 55.88 163.83 0)
+      (effects (font (size 1.27 1.27)) hide)
+    )
+    (property "Supplier Link" "" (at 55.88 163.83 0)
+      (effects (font (size 1.27 1.27)) hide)
+    )
+    (property "Part Number" "PESD3V3L1BA,115" (at 55.88 163.83 0)
+      (effects (font (size 1.27 1.27)) hide)
+    )
